Commit message: Added laser sensor

File: omni3ros_pkg/urdf/main.urdf.xacro (robot description, xacro)
@@ -33,4 +33,65 @@
 		<origin xyz="0 0 0.01905"/>
 	</joint>
+	<joint name="hokuyo_joint" type="fixed">
+	<axis xyz="0 1 0" />
+	<origin xyz=".15 0 .1" rpy="0 0 0"/>
+	<parent link="base_link"/>
+	<child link="hokuyo"/>
+	</joint>
+	<!-- Hokuyo Laser -->
+	<link name="hokuyo">
+	<collision>
+		<origin xyz="0 0 0" rpy="0 0 0"/>
+		<geometry>
+	<box size="0.1 0.1 0.1"/>
+		</geometry>
+	</collision>
+	<visual>
+		<origin xyz="0 0 0" rpy="0 0 0"/>
+		<geometry>
+		<mesh filename="package://omni3ros_pkg/mesh/hokuyo.dae"/>
+		</geometry>
+	</visual>
+	<inertial>
+		<mass value="1e-5" />
+		<origin xyz="0 0 0" rpy="0 0 0"/>
+		<inertia ixx="1e-6" ixy="0" ixz="0" iyy="1e-6" iyz="0" izz="1e-6" />
+	</inertial>
+	</link>
+	<gazebo reference="hokuyo">
+	<sensor type="ray" name="head_hokuyo_sensor">
+		<pose>0 0 0 0 0 0</pose>
+		<visualize>false</visualize>
+		<update_rate>40</update_rate>
+		<ray>
+		<scan>
+			<horizontal>
+			<samples>720</samples>
+			<resolution>1</resolution>
+			<min_angle>-1.570796</min_angle>
+			<max_angle>1.570796</max_angle>
+			</horizontal>
+		</scan>
+		<range>
+			<min>0.10</min>
+			<max>30.0</max>
+			<resolution>0.01</resolution>
+		</range>
+		<noise>
+			<type>gaussian</type>
+			<!-- Noise parameters based on published spec for Hokuyo laser
+				achieving "+-30mm" accuracy at range < 10m.  A mean of 0.0m and
+				stddev of 0.01m will put 99.7% of samples within 0.03m of the true
+				reading. -->
+			<mean>0.0</mean>
+			<stddev>0.01</stddev>
+		</noise>
+		</ray>
+		<plugin name="gazebo_ros_head_hokuyo_controller" filename="libgazebo_ros_laser.so">
+		<topicName>/scan</topicName>
+		<frameName>hokuyo</frameName>
+		</plugin>
+	</sensor>
+	</gazebo>
 	<xacro:rim_macro
 		name="left"

Commit message: Added gmapping support

File: omni3ros_pkg/urdf/main.urdf.xacro (robot description, xacro)
@@ -33,4 +33,31 @@
 		<origin xyz="0 0 0.01905"/>
 	</joint>
+	<xacro:rim_macro
+		name="left"
+		color="0.3 0 0"
+		xyz="-0.03464101615 0.02 0"
+		rpy="1.570796326794896 0 1.047197551196597"/>
+	<xacro:rim_macro
+		name="back"
+		color="0 0.3 0"
+		xyz="0 -0.04 0"
+		rpy="1.570796326794896 0 3.141592653589793"/>
+	<xacro:rim_macro
+		name="right"
+		color="0 0 0.3"
+		xyz="0.03464101615 0.02 0"
+		rpy="1.570796326794896 0 -1.047197551196597"/>
+	<gazebo reference="base_link">
+    		<material>Gazebo/White</material>
+  	</gazebo>
+	<gazebo reference="rim_left_link">
+    		<material>Gazebo/Red</material>
+  	</gazebo>
+	<gazebo reference="rim_back_link">
+    		<material>Gazebo/Green</material>
+  	</gazebo>
+	<gazebo reference="rim_right_link">
+    		<material>Gazebo/Blue</material>
+  	</gazebo>
 	<joint name="hokuyo_joint" type="fixed">
 	<axis xyz="0 1 0" />
@@ -94,31 +121,4 @@
 	</sensor>
 	</gazebo>
-	<xacro:rim_macro
-		name="left"
-		color="0.3 0 0"
-		xyz="-0.03464101615 0.02 0"
-		rpy="1.570796326794896 0 1.047197551196597"/>
-	<xacro:rim_macro
-		name="back"
-		color="0 0.3 0"
-		xyz="0 -0.04 0"
-		rpy="1.570796326794896 0 3.141592653589793"/>
-	<xacro:rim_macro
-		name="right"
-		color="0 0 0.3"
-		xyz="0.03464101615 0.02 0"
-		rpy="1.570796326794896 0 -1.047197551196597"/>
-	<gazebo reference="base_link">
-    		<material>Gazebo/White</material>
-  	</gazebo>
-	<gazebo reference="rim_left_link">
-    		<material>Gazebo/Red</material>
-  	</gazebo>
-	<gazebo reference="rim_back_link">
-    		<material>Gazebo/Green</material>
-  	</gazebo>
-	<gazebo reference="rim_right_link">
-    		<material>Gazebo/Blue</material>
-  	</gazebo>
 	<gazebo>
 		<plugin name="gazebo_ros_control" filename="libgazebo_ros_control.so">

Commit message: Added IMU and its fusion with wheel odometry with use of EKF

File: omni3ros_pkg/urdf/main.urdf.xacro (robot description, xacro)
@@ -2,35 +2,37 @@
 <robot xmlns:xacro="http://www.ros.org/wiki/xacro" name="open_base">
 	<xacro:include filename="$(find omni3ros_pkg)/urdf/rim.urdf.xacro"/>
-	<link name="origin_link"/>
+	<!-- <link name="origin_link"/> -->
 	<link name="base_link">
-	<inertial>
-		<mass value="0.07862944645"/>
-		<inertia
-			ixx="0.00002035985530754"
-			ixy="0"
-			ixz="0"
-			iyy="0.00002035985530754"
-			iyz="0"
-			izz="0.00003945961663220"/>
-		</inertial>
-	<visual>
-		<geometry>
-			<mesh filename="package://omni3ros_pkg/mesh/base.stl"/>
-		</geometry>
-		<material name="base_material">
-			<color rgba="1 1 1 1"/>
-		</material>
-	</visual>
-	<collision>
-		<geometry>
-			<mesh filename="package://omni3ros_pkg/mesh/base.stl"/>
-		</geometry>
-	</collision>
+		<inertial>
+			<!-- <mass value="0.07862944645"/> -->
+			<!-- Increased mass to decrease robot drift while standing -->
+			<mass value="0.07862944645"/>
+			<inertia
+				ixx="0.00002035985530754"
+				ixy="0"
+				ixz="0"
+				iyy="0.00002035985530754"
+				iyz="0"
+				izz="0.00003945961663220"/>
+			</inertial>
+		<visual>
+			<geometry>
+				<mesh filename="package://omni3ros_pkg/mesh/base.stl"/>
+			</geometry>
+			<material name="base_material">
+				<color rgba="1 1 1 1"/>
+			</material>
+		</visual>
+		<collision>
+			<geometry>
+				<mesh filename="package://omni3ros_pkg/mesh/base.stl"/>
+			</geometry>
+		</collision>
 	</link>
-	<joint name="base_joint" type="fixed">
+	<!-- <joint name="base_joint" type="fixed">
 		<parent link="origin_link" />
 		<child link="base_link" />
 		<origin xyz="0 0 0.01905"/>
-	</joint>
+	</joint> -->
 	<xacro:rim_macro
 		name="left"
@@ -62,5 +64,5 @@
 	<joint name="hokuyo_joint" type="fixed">
 	<axis xyz="0 1 0" />
-	<origin xyz=".15 0 .1" rpy="0 0 0"/>
+	<origin xyz="0 0 .04" rpy="0 0 0"/>
 	<parent link="base_link"/>
 	<child link="hokuyo"/>
@@ -96,6 +98,8 @@
 			<samples>720</samples>
 			<resolution>1</resolution>
-			<min_angle>-1.570796</min_angle>
-			<max_angle>1.570796</max_angle>
+			<!-- <min_angle>-1.570796</min_angle>
+			<max_angle>1.570796</max_angle> -->
+			<min_angle>-3.14159</min_angle>
+			<max_angle>3.14159</max_angle>
 			</horizontal>
 		</scan>
@@ -122,4 +126,27 @@
 	</gazebo>
 	<gazebo>
+		<plugin name="gazebo_ros_imu" filename="libgazebo_ros_imu.so">
+			<alwaysOn>true</alwaysOn>
+			<bodyName>base_link</bodyName>
+			<topicName>imu</topicName>
+			<serviceName>imu_service</serviceName>
+			<gaussianNoise>0.0</gaussianNoise>
+			<updateRate>50.0</updateRate>
+		</plugin>
+	</gazebo>
+	<!-- <gazebo>
+		<controller:gazebo_ros_imu name="imu_controller" plugin="libgazebo_ros_imu.so">
+			<alwaysOn>true</alwaysOn>
+			<updateRate>50.0</updateRate>
+			<bodyName>imu_link</bodyName>
+			<topicName>imu_data</topicName>
+			<gaussianNoise>2.89e-08</gaussianNoise>
+			<xyzOffsets>0 0 0</xyzOffsets>
+			<rpyOffsets>0 0 0</rpyOffsets>
+			<interface:position name="imu_position"/>
+		</controller:gazebo_ros_imu>
+	</gazebo> -->
+	<!-- ROS control -->
+	<gazebo>
 		<plugin name="gazebo_ros_control" filename="libgazebo_ros_control.so">
 		<robotNamespace>/open_base</robotNamespace>

Commit message: Added move_base package for path planning and control on the way to goal pose

File: omni3ros_pkg/urdf/main.urdf.xacro (robot description, xacro)
@@ -62,12 +62,12 @@
     		<material>Gazebo/Blue</material>
   	</gazebo>
-	<joint name="hokuyo_joint" type="fixed">
+	<joint name="laser_frame_joint" type="fixed">
 	<axis xyz="0 1 0" />
 	<origin xyz="0 0 .04" rpy="0 0 0"/>
 	<parent link="base_link"/>
-	<child link="hokuyo"/>
+	<child link="laser_frame"/>
 	</joint>
 	<!-- Hokuyo Laser -->
-	<link name="hokuyo">
+	<link name="laser_frame">
 	<collision>
 		<origin xyz="0 0 0" rpy="0 0 0"/>
@@ -88,5 +88,5 @@
 	</inertial>
 	</link>
-	<gazebo reference="hokuyo">
+	<gazebo reference="laser_frame">
 	<sensor type="ray" name="head_hokuyo_sensor">
 		<pose>0 0 0 0 0 0</pose>
@@ -121,5 +121,5 @@
 		<plugin name="gazebo_ros_head_hokuyo_controller" filename="libgazebo_ros_laser.so">
 		<topicName>/scan</topicName>
-		<frameName>hokuyo</frameName>
+		<frameName>laser_frame</frameName>
 		</plugin>
 	</sensor>

Commit message: Added sonar

File: omni3ros_pkg/urdf/main.urdf.xacro (robot description, xacro)
@@ -2,5 +2,5 @@
 <robot xmlns:xacro="http://www.ros.org/wiki/xacro" name="open_base">
 	<xacro:include filename="$(find omni3ros_pkg)/urdf/rim.urdf.xacro"/>
-	<!-- <link name="origin_link"/> -->
+	<xacro:arg name="sonar" default="false"/>
 	<link name="base_link">
 		<inertial>
@@ -30,9 +30,4 @@
 		</collision>
 	</link>
-	<!-- <joint name="base_joint" type="fixed">
-		<parent link="origin_link" />
-		<child link="base_link" />
-		<origin xyz="0 0 0.01905"/>
-	</joint> -->
 	<xacro:rim_macro
 		name="left"
@@ -62,67 +57,133 @@
     		<material>Gazebo/Blue</material>
   	</gazebo>
+	<!-- Hokuyo Laser -->
 	<joint name="laser_frame_joint" type="fixed">
-	<axis xyz="0 1 0" />
-	<origin xyz="0 0 .04" rpy="0 0 0"/>
-	<parent link="base_link"/>
-	<child link="laser_frame"/>
+		<axis xyz="0 1 0" />
+		<origin xyz="0 0 .04" rpy="0 0 0"/>
+		<parent link="base_link"/>
+		<child link="laser_frame"/>
 	</joint>
-	<!-- Hokuyo Laser -->
 	<link name="laser_frame">
-	<collision>
-		<origin xyz="0 0 0" rpy="0 0 0"/>
-		<geometry>
-	<box size="0.1 0.1 0.1"/>
-		</geometry>
-	</collision>
-	<visual>
-		<origin xyz="0 0 0" rpy="0 0 0"/>
-		<geometry>
-		<mesh filename="package://omni3ros_pkg/mesh/hokuyo.dae"/>
-		</geometry>
-	</visual>
-	<inertial>
-		<mass value="1e-5" />
-		<origin xyz="0 0 0" rpy="0 0 0"/>
-		<inertia ixx="1e-6" ixy="0" ixz="0" iyy="1e-6" iyz="0" izz="1e-6" />
-	</inertial>
+		<collision>
+			<origin xyz="0 0 0" rpy="0 0 0"/>
+			<geometry>
+				<box size="0.1 0.1 0.1"/>
+			</geometry>
+		</collision>
+		<visual>
+			<origin xyz="0 0 0" rpy="0 0 0"/>
+			<geometry>
+			<mesh filename="package://omni3ros_pkg/mesh/hokuyo.dae"/>
+			</geometry>
+		</visual>
+		<inertial>
+			<mass value="1e-5" />
+			<origin xyz="0 0 0" rpy="0 0 0"/>
+			<inertia ixx="1e-6" ixy="0" ixz="0" iyy="1e-6" iyz="0" izz="1e-6" />
+		</inertial>
 	</link>
 	<gazebo reference="laser_frame">
-	<sensor type="ray" name="head_hokuyo_sensor">
-		<pose>0 0 0 0 0 0</pose>
-		<visualize>false</visualize>
-		<update_rate>40</update_rate>
-		<ray>
-		<scan>
-			<horizontal>
-			<samples>720</samples>
-			<resolution>1</resolution>
-			<!-- <min_angle>-1.570796</min_angle>
-			<max_angle>1.570796</max_angle> -->
-			<min_angle>-3.14159</min_angle>
-			<max_angle>3.14159</max_angle>
-			</horizontal>
-		</scan>
-		<range>
-			<min>0.10</min>
-			<max>30.0</max>
-			<resolution>0.01</resolution>
-		</range>
-		<noise>
-			<type>gaussian</type>
-			<!-- Noise parameters based on published spec for Hokuyo laser
-				achieving "+-30mm" accuracy at range < 10m.  A mean of 0.0m and
-				stddev of 0.01m will put 99.7% of samples within 0.03m of the true
-				reading. -->
-			<mean>0.0</mean>
-			<stddev>0.01</stddev>
-		</noise>
-		</ray>
-		<plugin name="gazebo_ros_head_hokuyo_controller" filename="libgazebo_ros_laser.so">
-		<topicName>/scan</topicName>
-		<frameName>laser_frame</frameName>
-		</plugin>
-	</sensor>
+		<sensor type="ray" name="head_hokuyo_sensor">
+			<pose>0 0 0 0 0 0</pose>
+			<visualize>false</visualize>
+			<update_rate>40</update_rate>
+			<ray>
+			<scan>
+				<horizontal>
+				<samples>720</samples>
+				<resolution>1</resolution>
+				<!-- <min_angle>-1.570796</min_angle>
+				<max_angle>1.570796</max_angle> -->
+				<min_angle>-3.14159</min_angle>
+				<max_angle>3.14159</max_angle>
+				</horizontal>
+			</scan>
+			<range>
+				<min>0.10</min>
+				<max>30.0</max>
+				<resolution>0.01</resolution>
+			</range>
+			<noise>
+				<type>gaussian</type>
+				<!-- Noise parameters based on published spec for Hokuyo laser
+					achieving "+-30mm" accuracy at range < 10m.  A mean of 0.0m and
+					stddev of 0.01m will put 99.7% of samples within 0.03m of the true
+					reading. -->
+				<mean>0.0</mean>
+				<stddev>0.01</stddev>
+			</noise>
+			</ray>
+			<plugin name="gazebo_ros_head_hokuyo_controller" filename="libgazebo_ros_laser.so">
+			<topicName>/scan</topicName>
+			<frameName>laser_frame</frameName>
+			</plugin>
+		</sensor>
 	</gazebo>
+	<!-- Sonar -->
+	<xacro:if value="$(arg sonar)">
+		<joint name="sonar_frame_joint" type="fixed">
+			<axis xyz="0 1 0" />
+			<origin xyz="0 0 .1" rpy="0 0 0"/>
+			<parent link="base_link"/>
+			<child link="sonar_frame"/>
+		</joint>
+		<link name="sonar_frame">
+			<collision>
+				<origin xyz="0 0 0" rpy="0 0 0"/>
+				<geometry>
+					<box size="0.01 0.01 0.01"/>
+				</geometry>
+			</collision>
+			<visual>
+				<origin xyz="0 0 0" rpy="0 0 0"/>
+				<geometry>
+					<box size="0.01 0.01 0.01"/>
+				<!-- <mesh filename="package://omni3ros_pkg/mesh/hokuyo.dae"/> -->
+				</geometry>
+			</visual>
+			<inertial>
+				<mass value="1e-5" />
+				<origin xyz="0 0 0" rpy="0 0 0"/>
+				<inertia ixx="1e-6" ixy="0" ixz="0" iyy="1e-6" iyz="0" izz="1e-6" />
+			</inertial>
+		</link>
+		<gazebo reference="sonar_frame">
+			<sensor type="ray" name="TeraRanger">
+				<pose>0 0 0 0 0 0</pose>
+				<visualize>true</visualize>
+				<update_rate>50</update_rate>
+				<ray>
+					<scan>
+						<horizontal>
+						<samples>10</samples>
+						<resolution>1</resolution>
+						<min_angle>-0.14835</min_angle>
+						<max_angle>0.14835</max_angle>
+						</horizontal>
+						<vertical>
+						<samples>10</samples>
+						<resolution>1</resolution>
+						<min_angle>-0.14835</min_angle>
+						<max_angle>0.14835</max_angle>
+						</vertical>
+					</scan>
+					<range>
+						<min>0.01</min>
+						<max>2</max>
+						<resolution>0.02</resolution>
+					</range>
+				</ray>
+				<plugin filename="libgazebo_ros_range.so" name="gazebo_ros_range">
+					<!-- <gaussianNoise>0.005</gaussianNoise> -->
+					<alwaysOn>true</alwaysOn>
+					<updateRate>50</updateRate>
+					<topicName>sonar</topicName>
+					<frameName>sonar_frame</frameName>
+					<radiation>ultrasound</radiation>
+					<fov>0.2967</fov>
+				</plugin>
+			</sensor>
+		</gazebo>
+	</xacro:if>
 	<gazebo>
 		<plugin name="gazebo_ros_imu" filename="libgazebo_ros_imu.so">
@@ -135,16 +196,4 @@
 		</plugin>
 	</gazebo>
-	<!-- <gazebo>
-		<controller:gazebo_ros_imu name="imu_controller" plugin="libgazebo_ros_imu.so">
-			<alwaysOn>true</alwaysOn>
-			<updateRate>50.0</updateRate>
-			<bodyName>imu_link</bodyName>
-			<topicName>imu_data</topicName>
-			<gaussianNoise>2.89e-08</gaussianNoise>
-			<xyzOffsets>0 0 0</xyzOffsets>
-			<rpyOffsets>0 0 0</rpyOffsets>
-			<interface:position name="imu_position"/>
-		</controller:gazebo_ros_imu>
-	</gazebo> -->
 	<!-- ROS control -->
 	<gazebo>
