Commit message: Scaled platform to sizes of the real robot

File: omni3ros_pkg/urdf/model/rim.urdf.xacro (robot description, xacro)
@@ -1,5 +1,5 @@
 <?xml version="1.0" ?>
 <robot xmlns:xacro="http://www.ros.org/wiki/xacro">
-<xacro:include filename="$(find omni3ros_pkg)/urdf/roller.urdf.xacro"/>
+<xacro:include filename="$(find omni3ros_pkg)/urdf/model/roller.urdf.xacro"/>
 <xacro:macro
 	name="rim_macro"
@@ -10,14 +10,14 @@
 				<mass value="0.00835758"/>
 				<inertia
-					ixx="6.63684e-07"
+					ixx="6.63684e-04"
 					ixy="0"
 					ixz="0"
-					iyy="6.63684e-07"
+					iyy="6.63684e-04"
 					iyz="0"
-					izz="9.40333e-07"/>
+					izz="9.40333e-04"/>
 			</inertial>
 			<visual>
 				<geometry>
-					<mesh filename="package://omni3ros_pkg/mesh/rim.stl"/>
+					<mesh filename="package://omni3ros_pkg/mesh/model/rim.stl"/>
 				</geometry>
 				<material name="rim_${name}_material">
@@ -27,5 +27,5 @@
 			<collision>
 				<geometry>
-					<mesh filename="package://omni3ros_pkg/mesh/rim.stl"/>
+					<mesh filename="package://omni3ros_pkg/mesh/model/rim.stl"/>
 				</geometry>
 			</collision>
@@ -42,5 +42,5 @@
 			parent="${name}"
 			name="e"
-			xyz="0.01355 0 0.0055"
+			xyz="0.1355 0 0.055"
 			rpy="-1.570796326794896 0 0"
 		/>
@@ -48,5 +48,5 @@
 			parent="${name}"
 			name="ne"
-			xyz="0.00958129689 0.00958129689 -0.0055"
+			xyz="0.0958129689 0.0958129689 -0.0055"
 			rpy="-1.570796326794896 0 0.7853981633974483"
 		/>
@@ -54,5 +54,5 @@
 			parent="${name}"
 			name="n"
-			xyz="0 0.01355 0.0055"
+			xyz="0 0.1355 0.055"
 			rpy="-1.570796326794896 0 1.570796326794896"
 		/>
@@ -60,5 +60,5 @@
 			parent="${name}"
 			name="nw"
-			xyz="-0.00958129689 0.00958129689 -0.0055"
+			xyz="-0.0958129689 0.0958129689 -0.055"
 			rpy="-1.570796326794896 0 2.356194490192345"
 		/>
@@ -66,5 +66,5 @@
 			parent="${name}"
 			name="w"
-			xyz="-0.01355 0 0.0055"
+			xyz="-0.1355 0 0.055"
 			rpy="-1.570796326794896 0 3.141592653589793"
 		/>
@@ -72,5 +72,5 @@
 			parent="${name}"
 			name="sw"
-			xyz="-0.00958129689 -0.00958129689 -0.0055"
+			xyz="-0.0958129689 -0.0958129689 -0.055"
 			rpy="-1.570796326794896 0 -2.356194490192345"
 		/>
@@ -78,5 +78,5 @@
 			parent="${name}"
 			name="s"
-			xyz="0 -0.01355 0.0055"
+			xyz="0 -0.1355 0.055"
 			rpy="-1.570796326794896 0 -1.570796326794896"
 		/>
@@ -84,5 +84,5 @@
 			parent="${name}"
 			name="se"
-			xyz="0.00958129689 -0.00958129689 -0.0055"
+			xyz="0.0958129689 -0.0958129689 -0.055"
 			rpy="-1.570796326794896 0 -0.7853981633974483"
 		/>

File: omni3ros_pkg/urdf/model/roller.urdf.xacro (robot description, xacro)
@@ -8,14 +8,14 @@
 				<mass value="0.00113845"/>
 				<inertia
-					ixx="2.53776e-08"
+					ixx="2.53776e-05"
 					ixy="0"
 					ixz="0"
-					iyy="2.53776e-08"
+					iyy="2.53776e-05"
 					iyz="0"
-					izz="1.47666e-08"/>
+					izz="1.47666e-05"/>
 			</inertial>
 			<visual>
 				<geometry>
-					<mesh filename="package://omni3ros_pkg/mesh/roller.stl"/>
+					<mesh filename="package://omni3ros_pkg/mesh/model/roller.stl"/>
 				</geometry>
 				<material name="roller_material">
@@ -25,5 +25,5 @@
 			<collision>
 				<geometry>
-					<mesh filename="package://omni3ros_pkg/mesh/roller.stl"/>
+					<mesh filename="package://omni3ros_pkg/mesh/model/roller.stl"/>
 				</geometry>
 			</collision>
