Commit message: Added RGBD camera (kinnect)

File: omni3ros_pkg/urdf/model/main.urdf.xacro (robot description, xacro)
@@ -75,5 +75,5 @@
 				<origin xyz="0 0 0" rpy="0 0 0"/>
 				<geometry>
-				<mesh filename="package://omni3ros_pkg/mesh/hokuyo.dae"/>
+					<mesh filename="package://omni3ros_pkg/mesh/hokuyo.dae"/>
 				</geometry>
 			</visual>
@@ -106,5 +106,5 @@
 					</range>
 					<noise>
-						<type>gaussian</type>
+						<type>gaussian<mesh filename="package://omni3ros_pkg/mesh/hokuyo.dae"/></type>
 						<!-- Noise parameters based on published spec for Hokuyo laser
 							achieving "+-30mm" accuracy at range < 10m.  A mean of 0.0m and
@@ -158,19 +158,20 @@
 					<scan>
 						<horizontal>
-						<samples>10</samples>
-						<resolution>1</resolution>
-						<min_angle>-0.14835</min_angle>
-						<max_angle>0.14835</max_angle>
+							<samples>10</samples>
+							<resolution>1</resolution>
+							<min_angle>-0.14835</min_angle>
+							<max_angle>0.14835</max_angle>
 						</horizontal>
 						<vertical>
-						<samples>10</samples>
-						<resolution>1</resolution>
-						<min_angle>-0.14835</min_angle>
-						<max_angle>0.14835</max_angle>
+							<samples>10</samples>
+							<resolution>1</resolution>
+							<min_angle>-0.14835</min_angle>
+							<max_angle>0.14835</max_angle>
 						</vertical>
 					</scan>
 					<range>
 						<min>0.01</min>
-						<max>2</max>
+						<!-- TODO range is shown too small in the Gazebo and Rviz -->
+						<max>4</max>
 						<resolution>0.02</resolution>
 					</range>
@@ -189,49 +190,66 @@
 	</xacro:if>
 	<!-- RGBD Camera -->
-	<!-- Camera -->
-	<!-- <joint name="camera_joint" type="fixed">
-		<axis xyz="0 1 0" />
-		<origin xyz="0.05 0 0.2" rpy="0 0 0"/>
-		<parent link="base_link"/>
-		<child link="camera_link"/>
-  	</joint>
-	<link name="camera_link">
-		<collision>
-			<origin xyz="0 0 0" rpy="0 0 0"/>
-			<geometry>
-			<box size="0.05 0.05 0.05"/>
-			</geometry>
-		</collision>
-		<visual>
-			<origin xyz="0 0 0" rpy="0 0 0"/>
-			<geometry>
-			<box size="0.05 0.05 0.05"/>
-			</geometry>
-			<material name="red"/>
-		</visual>
-		<inertial>
-			<mass value="1e-5" />
-			<origin xyz="0 0 0" rpy="0 0 0"/>
-			<inertia ixx="1e-6" ixy="0" ixz="0" iyy="1e-6" iyz="0" izz="1e-6" />
-		</inertial>
-	</link>
-	<gazebo reference="camera_link">
-		<sensor name="depth_camera" type="depth">
-			<update_rate>20</update_rate>
-			<camera>
-				<horizontal_fov>1.047198</horizontal_fov>
-				<image>
-					<width>640</width>
-					<height>480</height>
-					<format>R8G8B8</format>
-				</image>
-				<clip>
-					<near>0.05</near>
-					<far>3</far>
-				</clip>
-			</camera>
-			<plugin name="camera_plugin" filename="libgazebo_ros_openni_kinect.so">
+	<!-- Intel realsense -->
+	<!-- <xacro:include filename="$(find omni3ros_pkg)/urdf/_d435.urdf.xacro"/> -->
+	<!-- <xacro:include filename="$(find omni3ros_pkg)/urdf/_d435.urdf.xacro">
+		<sensor_d435 parent="$base_link"></sensor_d435>
+	</xacro:include> -->
+	<!-- Kinnect -->
+	<xacro:if value="$(arg camera)">
+		<joint name="camera_frame_joint" type="fixed">
+			<axis xyz="0 1 0" />
+			<!-- 1.57 turned camera to look along y axis (it makes sense since now robot forward part looks at positive direction of y axis) -->
+			<origin xyz="0 0 .6" rpy="0 0 1.57"/>
+			<parent link="base_link"/>
+			<child link="camera_frame"/>
+		</joint>
+		<link name="camera_frame">
+			<collision name="collision">
+				<origin xyz="0 0 0" rpy="0 0 0"/>
+				<geometry>
+					<box size="0.073000 0.276000 0.072000"/>
+				</geometry>
+			</collision>
+			<visual name="visual">
+				<origin xyz="0 0 0" rpy="0 0 0"/>
+				<geometry>
+					<mesh filename="package://omni3ros_pkg/mesh/kinect.dae"/>
+				</geometry>
+			</visual>
+			<inertial>
+				<mass value="0.1" />
+				<origin xyz="0 0 0" rpy="0 0 0"/>
+				<inertia ixx="1e-6" ixy="0" ixz="0" iyy="1e-6" iyz="0" izz="1e-6" />
+			</inertial>
+		</link>
+		<!-- Need this since rviz frame does not match the kinects own frame. So for visualizing the kinect
+		model correctly in gazebo and rviz you need 1 transform, but to transform the data you need another.
+		https://answers.ros.org/question/329409/point-cloud-in-wrong-position-relative-to-robot/ -->
+		<joint name="camera_optical_joint" type="fixed">
+            <origin xyz="0 0 0" rpy="-1.5708 0 -1.5708"/>
+            <parent link="camera_frame"/>
+            <child link="camera_frame_optical"/>
+        </joint>
+        <link name="camera_frame_optical"/>
+		<gazebo reference="camera_frame">
+			<sensor type="depth" name="camera">
+				<update_rate>20</update_rate>
+				<camera>
+					<horizontal_fov>1.047198</horizontal_fov>
+					<image>
+						<width>640</width>
+						<height>480</height>
+						<format>R8G8B8</format>
+					</image>
+					<clip>
+						<near>0.05</near>
+						<far>3</far>
+					</clip>
+				</camera>
+				<plugin name="camera_plugin" filename="libgazebo_ros_openni_kinect.so">
 				<baseline>0.2</baseline>
 				<alwaysOn>true</alwaysOn>
+				<!-- Keep this zero, update_rate in the parent <sensor> tag
+					will control the frame rate. -->
 				<updateRate>0.0</updateRate>
 				<cameraName>camera_ir</cameraName>
@@ -241,5 +259,5 @@
 				<depthImageCameraInfoTopicName>/camera/depth/camera_info</depthImageCameraInfoTopicName>
 				<pointCloudTopicName>/camera/depth/points</pointCloudTopicName>
-				<frameName>camera_link</frameName>
+				<frameName>camera_frame_optical</frameName>
 				<pointCloudCutoff>0.5</pointCloudCutoff>
 				<pointCloudCutoffMax>3.0</pointCloudCutoffMax>
@@ -254,86 +272,9 @@
 				<focalLength>0</focalLength>
 				<hackBaseline>0</hackBaseline>
-			</plugin>
-		</sensor>
-	</gazebo> -->
-	<xacro:if value="$(arg camera)">
-		<joint name="camera_frame_joint" type="fixed">
-			<axis xyz="0 1 0" />
-			<origin xyz="0 0 .3" rpy="0 0 0"/>
-			<parent link="base_link"/>
-			<child link="camera_frame"/>
-		</joint>
-		<link name="camera_frame">
-			<inertial>
-				<mass value="1e-5" />
-				<origin xyz="0 0 0" rpy="0 0 0"/>
-				<inertia ixx="1e-6" ixy="0" ixz="0" iyy="1e-6" iyz="0" izz="1e-6" />
-			</inertial>
-			<collision name="collision">
-				<geometry>
-					<box>
-						<size>0.073000 0.276000 0.072000</size>
-					</box>
-				</geometry>
-			</collision>
-			<visual name="visual">
-				<!-- <geometry>
-					<mesh>
-						<uri>model://kinect_ros/meshes/kinect.dae</uri>
-						<uri>package://omni3ros_pkg/mesh/kinect.dae</uri>
-					</mesh>
-				</geometry> -->
-				<geometry>
-					<box>
-						<size>0.073000 0.276000 0.072000</size>
-					</box>
-      			</geometry>
-      			<material name="red"/>
-			</visual>
-		</link>
-		<gazebo reference="camera_frame">
-			<sensor name="camera" type="depth">
-				<update_rate>20</update_rate>
-				<camera>
-				<horizontal_fov>1.047198</horizontal_fov>
-				<image>
-					<width>640</width>
-					<height>480</height>
-					<format>R8G8B8</format>
-				</image>
-				<clip>
-					<near>0.05</near>
-					<far>3</far>
-				</clip>
-				</camera>
-				<plugin name="camera_plugin" filename="libgazebo_ros_camera.so">
-					<baseline>0.2</baseline>
-					<alwaysOn>true</alwaysOn>
-					<!-- Keep this zero, update_rate in the parent <sensor> tag
-						will control the frame rate. -->
-					<updateRate>0.0</updateRate>
-					<cameraName>camera_ir</cameraName>
-					<imageTopicName>/camera/color/image_raw</imageTopicName>
-					<cameraInfoTopicName>/camera/color/camera_info</cameraInfoTopicName>
-					<depthImageTopicName>/camera/depth/image_raw</depthImageTopicName>
-					<depthImageCameraInfoTopicName>/camera/depth/camera_info</depthImageCameraInfoTopicName>
-					<pointCloudTopicName>/camera/depth/points</pointCloudTopicName>
-					<frameName>camera_frame</frameName>
-					<pointCloudCutoff>0.5</pointCloudCutoff>
-					<pointCloudCutoffMax>3.0</pointCloudCutoffMax>
-					<distortionK1>0</distortionK1>
-					<distortionK2>0</distortionK2>
-					<distortionK3>0</distortionK3>
-					<distortionT1>0</distortionT1>
-					<distortionT2>0</distortionT2>
-					<CxPrime>0</CxPrime>
-					<Cx>0</Cx>
-					<Cy>0</Cy>
-					<focalLength>0</focalLength>
-					<hackBaseline>0</hackBaseline>
 				</plugin>
 			</sensor>
 		</gazebo>
 	</xacro:if>
+	<!-- IMU -->
 	<gazebo>
 		<plugin name="gazebo_ros_imu" filename="libgazebo_ros_imu.so">

Commit message: Rotated model layout (yaw), changed pitch of the camera

File: omni3ros_pkg/urdf/model/main.urdf.xacro (robot description, xacro)
@@ -7,5 +7,5 @@
 	<link name="base_link">
 		<inertial>
-			<mass value="0.17862944645"/>
+			<mass value="10.17862944645"/>
 			<inertia
 				ixx="0.002035985530754"
@@ -30,4 +30,5 @@
 		</collision>
 	</link>
+<!--
 	<xacro:rim_macro
 		name="left"
@@ -44,5 +45,20 @@
 		color="0 0 0.3"
 		xyz="0.3464101615 0.2 0"
-		rpy="1.570796326794896 0 -1.047197551196597"/>
+		rpy="1.570796326794896 0 -1.047197551196597"/> -->
+	<xacro:rim_macro
+		name="left"
+		color="0.3 0 0"
+		xyz="0.2 0.3464101615 0"
+		rpy="1.570796326794896 0 -0.523599"/>
+	<xacro:rim_macro
+		name="back"
+		color="0 0.3 0"
+		xyz="-0.4 0 0"
+		rpy="1.570796326794896 0 1.5708"/>
+	<xacro:rim_macro
+		name="right"
+		color="0 0 0.3"
+		xyz="0.2 -0.3464101615 0"
+		rpy="1.570796326794896 0 -2.61799"/>
 	<gazebo reference="base_link">
     		<material>Gazebo/White</material>
@@ -199,6 +215,6 @@
 		<joint name="camera_frame_joint" type="fixed">
 			<axis xyz="0 1 0" />
-			<!-- 1.57 turned camera to look along y axis (it makes sense since now robot forward part looks at positive direction of y axis) -->
-			<origin xyz="0 0 .6" rpy="0 0 1.57"/>
+			<!-- Positive pitch so camera looks downwards to see ground obstacles -->
+			<origin xyz="0 0 .6" rpy="0 0.25 0"/>
 			<parent link="base_link"/>
 			<child link="camera_frame"/>
@@ -242,34 +258,35 @@
 						<format>R8G8B8</format>
 					</image>
-					<clip>
+					<!-- In default setup it was turned on, however it's doesn't make sense  -->
+					<!-- <clip>
 						<near>0.05</near>
 						<far>3</far>
-					</clip>
+					</clip> -->
 				</camera>
 				<plugin name="camera_plugin" filename="libgazebo_ros_openni_kinect.so">
-				<baseline>0.2</baseline>
-				<alwaysOn>true</alwaysOn>
-				<!-- Keep this zero, update_rate in the parent <sensor> tag
-					will control the frame rate. -->
-				<updateRate>0.0</updateRate>
-				<cameraName>camera_ir</cameraName>
-				<imageTopicName>/camera/color/image_raw</imageTopicName>
-				<cameraInfoTopicName>/camera/color/camera_info</cameraInfoTopicName>
-				<depthImageTopicName>/camera/depth/image_raw</depthImageTopicName>
-				<depthImageCameraInfoTopicName>/camera/depth/camera_info</depthImageCameraInfoTopicName>
-				<pointCloudTopicName>/camera/depth/points</pointCloudTopicName>
-				<frameName>camera_frame_optical</frameName>
-				<pointCloudCutoff>0.5</pointCloudCutoff>
-				<pointCloudCutoffMax>3.0</pointCloudCutoffMax>
-				<distortionK1>0</distortionK1>
-				<distortionK2>0</distortionK2>
-				<distortionK3>0</distortionK3>
-				<distortionT1>0</distortionT1>
-				<distortionT2>0</distortionT2>
-				<CxPrime>0</CxPrime>
-				<Cx>0</Cx>
-				<Cy>0</Cy>
-				<focalLength>0</focalLength>
-				<hackBaseline>0</hackBaseline>
+					<baseline>0.2</baseline>
+					<alwaysOn>true</alwaysOn>
+					<!-- Keep this zero, update_rate in the parent <sensor> tag
+						will control the frame rate. -->
+					<updateRate>0.0</updateRate>
+					<cameraName>camera_ir</cameraName>
+					<imageTopicName>/camera/color/image_raw</imageTopicName>
+					<cameraInfoTopicName>/camera/color/camera_info</cameraInfoTopicName>
+					<depthImageTopicName>/camera/depth/image_raw</depthImageTopicName>
+					<depthImageCameraInfoTopicName>/camera/depth/camera_info</depthImageCameraInfoTopicName>
+					<pointCloudTopicName>/camera/depth/points</pointCloudTopicName>
+					<frameName>camera_frame_optical</frameName>
+					<pointCloudCutoff>0.5</pointCloudCutoff>
+					<pointCloudCutoffMax>3.0</pointCloudCutoffMax>
+					<distortionK1>0</distortionK1>
+					<distortionK2>0</distortionK2>
+					<distortionK3>0</distortionK3>
+					<distortionT1>0</distortionT1>
+					<distortionT2>0</distortionT2>
+					<CxPrime>0</CxPrime>
+					<Cx>0</Cx>
+					<Cy>0</Cy>
+					<focalLength>0</focalLength>
+					<hackBaseline>0</hackBaseline>
 				</plugin>
 			</sensor>

Commit message: Added second 2D lidar

File: omni3ros_pkg/urdf/model/main.urdf.xacro (robot description, xacro)
@@ -2,4 +2,5 @@
 <robot xmlns:xacro="http://www.ros.org/wiki/xacro" name="open_base">
 	<xacro:include filename="$(find omni3ros_pkg)/urdf/model/rim.urdf.xacro"/>
+	<xacro:include filename="$(find omni3ros_pkg)/urdf/model/laser.urdf.xacro"/>
 	<xacro:arg name="sonar" default="false"/>
 	<xacro:arg name="lidar" default="true"/>
@@ -62,79 +63,61 @@
 		rpy="1.570796326794896 0 -2.61799"/>
 	<gazebo reference="base_link">
-    		<material>Gazebo/White</material>
+    		<material>Gazebo/Gray</material>
   	</gazebo>
 	<gazebo reference="rim_left_link">
-    		<material>Gazebo/Red</material>
+    		<material>Gazebo/Black</material>
   	</gazebo>
 	<gazebo reference="rim_back_link">
-    		<material>Gazebo/Green</material>
+    		<material>Gazebo/Black</material>
   	</gazebo>
 	<gazebo reference="rim_right_link">
-    		<material>Gazebo/Blue</material>
+    		<material>Gazebo/Black</material>
+  	</gazebo>
+	<!-- Chair -->
+	<joint name="chair_joint" type="fixed">
+		<axis xyz="0 1 0" />
+		<origin xyz="0 0 0" rpy="0 0 1.57"/>
+		<parent link="base_link"/>
+		<child link="chair_frame"/>
+	</joint>
+	<link name="chair_frame">
+		<collision>
+			<origin xyz="0 0 0.7" rpy="0 0 0"/>
+			<geometry>
+				<box size="0.8 0.6 0.8"/>
+			</geometry>
+		</collision>
+		<visual>
+			<origin xyz="0 0 0" rpy="0 0 0"/>
+			<geometry>
+				<mesh filename="package://omni3ros_pkg/mesh/model/office_chair.stl"/>
+			</geometry>
+		</visual>
+		<inertial>
+			<mass value="1e-5" />
+			<origin xyz="0 0 0" rpy="0 0 0"/>
+			<inertia ixx="1e-6" ixy="0" ixz="0" iyy="1e-6" iyz="0" izz="1e-6" />
+		</inertial>
+	</link>
+	<gazebo reference="chair_frame">
+    		<material>Gazebo/Gray</material>
   	</gazebo>
 	<!-- Hokuyo Laser -->
 	<xacro:if value="$(arg lidar)">
-		<joint name="laser_frame_joint" type="fixed">
-			<axis xyz="0 1 0" />
-			<origin xyz="0 0 .3" rpy="0 0 0"/>
-			<parent link="base_link"/>
-			<child link="laser_frame"/>
-		</joint>
-		<link name="laser_frame">
-			<collision>
-				<origin xyz="0 0 0" rpy="0 0 0"/>
-				<geometry>
-					<box size="0.1 0.1 0.1"/>
-				</geometry>
-			</collision>
-			<visual>
-				<origin xyz="0 0 0" rpy="0 0 0"/>
-				<geometry>
-					<mesh filename="package://omni3ros_pkg/mesh/hokuyo.dae"/>
-				</geometry>
-			</visual>
-			<inertial>
-				<mass value="1e-5" />
-				<origin xyz="0 0 0" rpy="0 0 0"/>
-				<inertia ixx="1e-6" ixy="0" ixz="0" iyy="1e-6" iyz="0" izz="1e-6" />
-			</inertial>
-		</link>
-		<gazebo reference="laser_frame">
-			<sensor type="gpu_ray" name="head_hokuyo_sensor">
-				<pose>0 0 0 0 0 0</pose>
-				<visualize>false</visualize>
-				<update_rate>40</update_rate>
-				<ray>
-					<scan>
-						<horizontal>
-						<samples>720</samples>
-						<resolution>1</resolution>
-						<!-- <min_angle>-1.570796</min_angle>
-						<max_angle>1.570796</max_angle> -->
-						<min_angle>-3.14159</min_angle>
-						<max_angle>3.14159</max_angle>
-						</horizontal>
-					</scan>
-					<range>
-						<min>0.10</min>
-						<max>30.0</max>
-						<resolution>0.01</resolution>
-					</range>
-					<noise>
-						<type>gaussian<mesh filename="package://omni3ros_pkg/mesh/hokuyo.dae"/></type>
-						<!-- Noise parameters based on published spec for Hokuyo laser
-							achieving "+-30mm" accuracy at range < 10m.  A mean of 0.0m and
-							stddev of 0.01m will put 99.7% of samples within 0.03m of the true
-							reading. -->
-						<mean>0.0</mean>
-						<stddev>0.01</stddev>
-					</noise>
-				</ray>
-				<plugin name="gazebo_ros_head_hokuyo_controller" filename="libgazebo_ros_gpu_laser.so">
-				<topicName>/scan</topicName>
-				<frameName>laser_frame</frameName>
-				</plugin>
-			</sensor>
-		</gazebo>
+		<!-- <xacro:laser
+			name=""
+			xyz="0 0 1.3"/> -->
+		<xacro:laser
+			name="_left"
+			xyz="0.15 0.35 .6"/>
+		<xacro:laser
+			name="_right"
+			xyz="0.15 -0.35 .6"/>
+		<joint name="laser_frame_merged_joint" type="fixed">
+            <origin xyz="0.15 0 0.6" rpy="0 0 0"/>
+            <parent link="base_link"/>
+            <child link="laser_frame_merged"/>
+        </joint>
+        <link name="laser_frame_merged"/>
 	</xacro:if>
 	<!-- Sonar -->

Commit message: Fixed model drifting

File: omni3ros_pkg/urdf/model/main.urdf.xacro (robot description, xacro)
@@ -9,11 +9,11 @@
 			<mass value="10.17862944645"/>
 			<inertia
-				ixx="0.002035985530754"
+				ixx="0.2035985530754"
 				ixy="0"
 				ixz="0"
-				iyy="0.002035985530754"
+				iyy="0.2035985530754"
 				iyz="0"
-				izz="0.003945961663220"/>
-			</inertial>
+				izz="0.3945961663220"/>
+		</inertial>
 		<visual>
 			<geometry>
