Commit message: Changed platform model

File: omni3ros_pkg/urdf/model_old/main.urdf.xacro (robot description, xacro)
@@ -30,19 +30,35 @@
 		</collision>
 	</link>
+<!--
 	<xacro:rim_macro
 		name="left"
 		color="0.3 0 0"
-		xyz="0.236282 0.260128 0"
-		rpy="1.570796326794896 0 -2.094399"/>
+		xyz="-0.3464101615 0.2 0"
+		rpy="1.570796326794896 0 1.047197551196597"/>
 	<xacro:rim_macro
 		name="back"
 		color="0 0.3 0"
-		xyz="-0.31 0.08 0"
-		rpy="1.570796326794896 0 0"/>
+		xyz="0 -0.4 0"
+		rpy="1.570796326794896 0 3.141592653589793"/>
 	<xacro:rim_macro
 		name="right"
 		color="0 0 0.3"
-		xyz="0.067718 -0.307128 0"
-		rpy="1.570796326794896 0 -4.18879"/>
+		xyz="0.3464101615 0.2 0"
+		rpy="1.570796326794896 0 -1.047197551196597"/> -->
+	<xacro:rim_macro
+		name="left"
+		color="0.3 0 0"
+		xyz="0.2 0.3464101615 0"
+		rpy="1.570796326794896 0 -0.523599"/>
+	<xacro:rim_macro
+		name="back"
+		color="0 0.3 0"
+		xyz="-0.4 0 0"
+		rpy="1.570796326794896 0 1.5708"/>
+	<xacro:rim_macro
+		name="right"
+		color="0 0 0.3"
+		xyz="0.2 -0.3464101615 0"
+		rpy="1.570796326794896 0 -2.61799"/>
 	<gazebo reference="base_link">
     		<material>Gazebo/White</material>

File: omni3ros_pkg/urdf/model_old/rim.urdf.xacro (robot description, xacro)
@@ -8,5 +8,5 @@
 			<inertial>
 				<origin xyz="0 0 -0.000343"/>
-				<mass value="0.0835758"/>
+				<mass value="0.00835758"/>
 				<inertia
 					ixx="6.63684e-04"
@@ -42,5 +42,5 @@
 			parent="${name}"
 			name="e"
-			xyz="0.0813 0 0.033"
+			xyz="0.1355 0 0.055"
 			rpy="-1.570796326794896 0 0"
 		/>
@@ -48,5 +48,5 @@
 			parent="${name}"
 			name="ne"
-			xyz="0.05748778 0.05748778 -0.033"
+			xyz="0.0958129689 0.0958129689 -0.055"
 			rpy="-1.570796326794896 0 0.7853981633974483"
 		/>
@@ -54,5 +54,5 @@
 			parent="${name}"
 			name="n"
-			xyz="0 0.0813 0.033"
+			xyz="0 0.1355 0.055"
 			rpy="-1.570796326794896 0 1.570796326794896"
 		/>
@@ -60,5 +60,5 @@
 			parent="${name}"
 			name="nw"
-			xyz="-0.05748778 0.05748778 -0.033"
+			xyz="-0.0958129689 0.0958129689 -0.055"
 			rpy="-1.570796326794896 0 2.356194490192345"
 		/>
@@ -66,5 +66,5 @@
 			parent="${name}"
 			name="w"
-			xyz="-0.0813 0 0.033"
+			xyz="-0.1355 0 0.055"
 			rpy="-1.570796326794896 0 3.141592653589793"
 		/>
@@ -72,5 +72,5 @@
 			parent="${name}"
 			name="sw"
-			xyz="-0.05748778 -0.05748778 -0.033"
+			xyz="-0.0958129689 -0.0958129689 -0.055"
 			rpy="-1.570796326794896 0 -2.356194490192345"
 		/>
@@ -78,5 +78,5 @@
 			parent="${name}"
 			name="s"
-			xyz="0 -0.0813 0.033"
+			xyz="0 -0.1355 0.055"
 			rpy="-1.570796326794896 0 -1.570796326794896"
 		/>
@@ -84,5 +84,5 @@
 			parent="${name}"
 			name="se"
-			xyz="0.05748778 -0.05748778 -0.033"
+			xyz="0.0958129689 -0.0958129689 -0.055"
 			rpy="-1.570796326794896 0 -0.7853981633974483"
 		/>

File: omni3ros_pkg/urdf/model_old/roller.urdf.xacro (robot description, xacro)
@@ -6,5 +6,5 @@
 		<link name="roller_${name}_rim_${parent}_link">
 			<inertial>
-				<mass value="0.0113845"/>
+				<mass value="0.00113845"/>
 				<inertia
 					ixx="2.53776e-05"
