Commit message: Refactored robot model version folders

File: omni3ros_pkg/urdf/model_ver3/main.urdf.xacro (robot description, xacro)
@@ -1,6 +1,6 @@
 <?xml version="1.0"?>
 <robot xmlns:xacro="http://www.ros.org/wiki/xacro" name="open_base">
-	<xacro:include filename="$(find omni3ros_pkg)/urdf/model/rim.urdf.xacro"/>
-	<xacro:include filename="$(find omni3ros_pkg)/urdf/model/laser.urdf.xacro"/>
+	<xacro:include filename="$(find omni3ros_pkg)/urdf/model_ver3/rim.urdf.xacro"/>
+	<xacro:include filename="$(find omni3ros_pkg)/urdf/model_ver3/laser.urdf.xacro"/>
 	<xacro:arg name="sonar" default="false"/>
 	<xacro:arg name="lidar" default="true"/>
@@ -19,5 +19,5 @@
 		<visual>
 			<geometry>
-				<mesh filename="package://omni3ros_pkg/mesh/model/base.stl"/>
+				<mesh filename="package://omni3ros_pkg/mesh/model_ver3/base.stl"/>
 			</geometry>
 			<material name="base_material">
@@ -27,5 +27,5 @@
 		<collision>
 			<geometry>
-				<mesh filename="package://omni3ros_pkg/mesh/model/base.stl"/>
+				<mesh filename="package://omni3ros_pkg/mesh/model_ver3/base.stl"/>
 			</geometry>
 		</collision>
@@ -75,5 +75,5 @@
 			<origin xyz="0 0 0" rpy="0 0 0"/>
 			<geometry>
-				<mesh filename="package://omni3ros_pkg/mesh/model/office_chair.stl"/>
+				<mesh filename="package://omni3ros_pkg/mesh/model_ver3/office_chair.stl"/>
 			</geometry>
 		</visual>

File: omni3ros_pkg/urdf/model_ver3/rim.urdf.xacro (robot description, xacro)
@@ -1,5 +1,5 @@
 <?xml version="1.0" ?>
 <robot xmlns:xacro="http://www.ros.org/wiki/xacro">
-<xacro:include filename="$(find omni3ros_pkg)/urdf/model/roller.urdf.xacro"/>
+<xacro:include filename="$(find omni3ros_pkg)/urdf/model_ver3/roller.urdf.xacro"/>
 <xacro:macro
 	name="rim_macro"
@@ -19,5 +19,5 @@
 			<visual>
 				<geometry>
-					<mesh filename="package://omni3ros_pkg/mesh/model/rim.stl"/>
+					<mesh filename="package://omni3ros_pkg/mesh/model_ver3/rim.stl"/>
 				</geometry>
 				<material name="rim_${name}_material">
@@ -27,5 +27,5 @@
 			<collision>
 				<geometry>
-					<mesh filename="package://omni3ros_pkg/mesh/model/rim.stl"/>
+					<mesh filename="package://omni3ros_pkg/mesh/model_ver3/rim.stl"/>
 				</geometry>
 			</collision>

File: omni3ros_pkg/urdf/model_ver3/roller.urdf.xacro (robot description, xacro)
@@ -17,5 +17,5 @@
 			<visual>
 				<geometry>
-					<mesh filename="package://omni3ros_pkg/mesh/model/roller.stl"/>
+					<mesh filename="package://omni3ros_pkg/mesh/model_ver3/roller.stl"/>
 				</geometry>
 				<material name="roller_material">
@@ -25,5 +25,5 @@
 			<collision>
 				<geometry>
-					<mesh filename="package://omni3ros_pkg/mesh/model/roller.stl"/>
+					<mesh filename="package://omni3ros_pkg/mesh/model_ver3/roller.stl"/>
 				</geometry>
 			</collision>
