Commit message: Refactored robot model version folders

File: omni3ros_pkg/urdf/model_ver2/main.urdf.xacro (robot description, xacro)
@@ -1,6 +1,6 @@
 <?xml version="1.0"?>
 <robot xmlns:xacro="http://www.ros.org/wiki/xacro" name="open_base">
-	<xacro:include filename="$(find omni3ros_pkg)/urdf/model/rim.urdf.xacro"/>
-	<xacro:include filename="$(find omni3ros_pkg)/urdf/model/laser.urdf.xacro"/>
+	<xacro:include filename="$(find omni3ros_pkg)/urdf/model_ver2/rim.urdf.xacro"/>
+	<xacro:include filename="$(find omni3ros_pkg)/urdf/model_ver2/laser.urdf.xacro"/>
 	<xacro:arg name="sonar" default="false"/>
 	<xacro:arg name="lidar" default="true"/>
@@ -19,5 +19,5 @@
 		<visual>
 			<geometry>
-				<mesh filename="package://omni3ros_pkg/mesh/model/base.stl"/>
+				<mesh filename="package://omni3ros_pkg/mesh/model_ver2/base.stl"/>
 			</geometry>
 			<material name="base_material">
@@ -27,5 +27,5 @@
 		<collision>
 			<geometry>
-				<mesh filename="package://omni3ros_pkg/mesh/model/base.stl"/>
+				<mesh filename="package://omni3ros_pkg/mesh/model_ver2/base.stl"/>
 			</geometry>
 		</collision>
@@ -91,5 +91,5 @@
 			<origin xyz="0 0 0" rpy="0 0 0"/>
 			<geometry>
-				<mesh filename="package://omni3ros_pkg/mesh/model/office_chair.stl"/>
+				<mesh filename="package://omni3ros_pkg/mesh/model_ver2/office_chair.stl"/>
 			</geometry>
 		</visual>

File: omni3ros_pkg/urdf/model_ver2/rim.urdf.xacro (robot description, xacro)
@@ -1,5 +1,5 @@
 <?xml version="1.0" ?>
 <robot xmlns:xacro="http://www.ros.org/wiki/xacro">
-<xacro:include filename="$(find omni3ros_pkg)/urdf/model/roller.urdf.xacro"/>
+<xacro:include filename="$(find omni3ros_pkg)/urdf/model_ver2/roller.urdf.xacro"/>
 <xacro:macro
 	name="rim_macro"
@@ -19,5 +19,5 @@
 			<visual>
 				<geometry>
-					<mesh filename="package://omni3ros_pkg/mesh/model/rim.stl"/>
+					<mesh filename="package://omni3ros_pkg/mesh/model_ver2/rim.stl"/>
 				</geometry>
 				<material name="rim_${name}_material">
@@ -27,5 +27,5 @@
 			<collision>
 				<geometry>
-					<mesh filename="package://omni3ros_pkg/mesh/model/rim.stl"/>
+					<mesh filename="package://omni3ros_pkg/mesh/model_ver2/rim.stl"/>
 				</geometry>
 			</collision>

Commit message: Finished merge branch 'chair' into devel

File: omni3ros_pkg/urdf/model_ver2/main.urdf.xacro (robot description, xacro)
@@ -2,4 +2,5 @@
 <robot xmlns:xacro="http://www.ros.org/wiki/xacro" name="open_base">
 	<xacro:include filename="$(find omni3ros_pkg)/urdf/model_ver2/rim.urdf.xacro"/>
+	<xacro:include filename="$(find omni3ros_pkg)/urdf/model_ver2/laser.urdf.xacro"/>
 	<xacro:arg name="sonar" default="false"/>
 	<xacro:arg name="lidar" default="true"/>
@@ -57,4 +58,51 @@
     		<material>Gazebo/Blue</material>
   	</gazebo>
+	<!-- Chair -->
+	<joint name="chair_joint" type="fixed">
+		<axis xyz="0 1 0" />
+		<origin xyz="0 0 0" rpy="0 0 1.57"/>
+		<parent link="base_link"/>
+		<child link="chair_frame"/>
+	</joint>
+	<link name="chair_frame">
+		<collision>
+			<origin xyz="0 0 0.7" rpy="0 0 0"/>
+			<geometry>
+				<box size="0.8 0.6 0.8"/>
+			</geometry>
+		</collision>
+		<visual>
+			<origin xyz="0 0 0" rpy="0 0 0"/>
+			<geometry>
+				<mesh filename="package://omni3ros_pkg/mesh/model_ver2/office_chair.stl"/>
+			</geometry>
+		</visual>
+		<inertial>
+			<mass value="1e-5" />
+			<origin xyz="0 0 0" rpy="0 0 0"/>
+			<inertia ixx="1e-6" ixy="0" ixz="0" iyy="1e-6" iyz="0" izz="1e-6" />
+		</inertial>
+	</link>
+	<gazebo reference="chair_frame">
+    		<material>Gazebo/Gray</material>
+  	</gazebo>
+	<!-- Hokuyo Laser -->
+	<xacro:if value="$(arg lidar)">
+		<!-- <xacro:laser
+			name=""
+			xyz="0 0 1.3"/> -->
+		<xacro:laser
+			name="_left"
+			xyz="0.15 0.35 .6"/>
+		<xacro:laser
+			name="_right"
+			xyz="0.15 -0.35 .6"/>
+		<joint name="laser_frame_merged_joint" type="fixed">
+            <origin xyz="0.15 0 0.6" rpy="0 0 0"/>
+            <parent link="base_link"/>
+            <child link="laser_frame_merged"/>
+        </joint>
+        <link name="laser_frame_merged"/>
+	</xacro:if>
 	<!-- Sonar -->
 	<xacro:if value="$(arg sonar)">
@@ -230,49 +278,2 @@
 	</gazebo>
 </robot>
-	<!-- Chair -->
-	<joint name="chair_joint" type="fixed">
-		<axis xyz="0 1 0" />
-		<origin xyz="0 0 0" rpy="0 0 1.57"/>
-		<parent link="base_link"/>
-		<child link="chair_frame"/>
-	</joint>
-	<link name="chair_frame">
-		<collision>
-			<origin xyz="0 0 0.7" rpy="0 0 0"/>
-			<geometry>
-				<box size="0.8 0.6 0.8"/>
-			</geometry>
-		</collision>
-		<visual>
-			<origin xyz="0 0 0" rpy="0 0 0"/>
-			<geometry>
-				<mesh filename="package://omni3ros_pkg/mesh/model_ver2/office_chair.stl"/>
-			</geometry>
-		</visual>
-		<inertial>
-			<mass value="1e-5" />
-			<origin xyz="0 0 0" rpy="0 0 0"/>
-			<inertia ixx="1e-6" ixy="0" ixz="0" iyy="1e-6" iyz="0" izz="1e-6" />
-		</inertial>
-	</link>
-	<gazebo reference="chair_frame">
-    		<material>Gazebo/Gray</material>
-  	</gazebo>
-	<!-- Hokuyo Laser -->
-	<xacro:if value="$(arg lidar)">
-		<!-- <xacro:laser
-			name=""
-			xyz="0 0 1.3"/> -->
-		<xacro:laser
-			name="_left"
-			xyz="0.15 0.35 .6"/>
-		<xacro:laser
-			name="_right"
-			xyz="0.15 -0.35 .6"/>
-		<joint name="laser_frame_merged_joint" type="fixed">
-            <origin xyz="0.15 0 0.6" rpy="0 0 0"/>
-            <parent link="base_link"/>
-            <child link="laser_frame_merged"/>
-        </joint>
-        <link name="laser_frame_merged"/>
-	</xacro:if>

Commit message: Converted depth camera's point cloud to laserscan and merged with others

File: omni3ros_pkg/urdf/model_ver2/main.urdf.xacro (robot description, xacro)
@@ -183,5 +183,5 @@
 			<axis xyz="0 1 0" />
 			<!-- Positive pitch so camera looks downwards to see ground obstacles -->
-			<origin xyz="0 0 .6" rpy="0 0.25 0"/>
+			<origin xyz="0.2 -0.15 .6" rpy="0 0.25 0"/>
 			<parent link="base_link"/>
 			<child link="camera_frame"/>
@@ -245,5 +245,6 @@
 					<frameName>camera_frame_optical</frameName>
 					<pointCloudCutoff>0.5</pointCloudCutoff>
-					<pointCloudCutoffMax>3.0</pointCloudCutoffMax>
+					<!-- We cut point cloud also when converting point cloud to laserscans (parameters are in camera_to_scan.launch) -->
+					<pointCloudCutoffMax>3.5</pointCloudCutoffMax>
 					<distortionK1>0</distortionK1>
 					<distortionK2>0</distortionK2>
